Commit message: WIP teleop

File: assets/objects/t_object.urdf (robot description, URDF)
Before this commit: robot t_object, 1 links, 0 joints
Links:
- removed link base
- added link crossbar, mass 0.5; collision box size=0.15 0.05 0.05; visual box size=0.15 0.05 0.05
- added link stem, mass 0.5; collision box size=0.05 0.10 0.05; visual box size=0.05 0.10 0.05
Joints:
- added joint stem_to_crossbar: type fixed, parent stem, child crossbar, origin xyz=0 0 0 rpy=0 0 0

Commit message: cleanup

File: assets/objects/t_object.urdf (robot description, URDF)
Before this commit: robot t_object, 2 links, 1 joints
Links:
- removed link crossbar
- removed link stem
- added link base, mass 1.0; collision box size=0.05 0.10 0.05; collision box size=0.15 0.05 0.05
Joints:
- removed joint stem_to_crossbar
